File: out/bluebuzz-rm2.kicad_sch (KiCad schematic)
At the start: 109 parts, among them J1 USB-C, J2 BAT, J3 SWD, J4 MOT, J5 TP, J6 PROBE, Q1 AO3400A, Q2 AO3400A, Q3 2N7002, SW1 PWR, U1 RP2350A, U10 USBLC6-2P6, U11 TPS22918DBVR, U2 BQ24074RGT, U20 DPS368, U21 DPS368, U22 DPS368, U23 DPS368, U24 DPS368, U3 TLV75533PDBV, U30 LSM6DS3TR-C, U5 TPS22918DBVR, U6 W25Q32JVUUIQ, U7 RM2, Y1 12MHz

Commit message: Routing gate review: failed; add parity, current and plane checks
design/gates/phase7.md records the gate. DRC is 0/0 and connectivity
parity is clean, but every high-current layer change is a single via,
the In3 VSYS pour is cut in two by signal wiring, and return vias and
edge stitching are missing. It holds the evidence, the independent
review's findings and the fix plan.

New checks: scripts/check_parity.py (schematic vs board by pad sets),
scripts/check_current.py (max-flow of each power path against the
design currents), scripts/check_planes.py (plane pieces and voids,
fast nets over their reference, return vias).

The schematic now carries the board's BOM/DNP flags (circuit.DNP).

Co-Authored-By: Claude Opus 5.5 <noreply@anthropic.com>
Parts:
- J2, J3, J4, J5: now left out of the parts list
- J6: now not fitted; now left out of the parts list
Changed lines of the file:
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@@
 	(symbol (lib_id "gen:pads_bat")
 		(at 172.72 284.48 0)
-		(unit 1) (exclude_from_sim no) (in_bom yes) (on_board yes) (dnp no)
+		(unit 1) (exclude_from_sim no) (in_bom no) (on_board yes) (dnp no)
 		(property "Reference" "J2" (at 162.56 275.26 0)
 			(effects (font (size 1.27 1.27)) (justify left bottom)))
@@
 	(symbol (lib_id "gen:pads_swd")
 		(at 238.76 241.3 0)
-		(unit 1) (exclude_from_sim no) (in_bom yes) (on_board yes) (dnp no)
+		(unit 1) (exclude_from_sim no) (in_bom no) (on_board yes) (dnp no)
 		(property "Reference" "J3" (at 228.6 229.54 0)
 			(effects (font (size 1.27 1.27)) (justify left bottom)))
@@
 	(symbol (lib_id "gen:debug_jst")
 		(at 238.76 292.1 0)
-		(unit 1) (exclude_from_sim no) (in_bom yes) (on_board yes) (dnp no)
+		(unit 1) (exclude_from_sim no) (in_bom no) (on_board yes) (dnp yes)
 		(property "Reference" "J6" (at 228.6 282.88 0)
 			(effects (font (size 1.27 1.27)) (justify left bottom)))
@@
 	(symbol (lib_id "gen:pads_tp")
 		(at 238.76 266.7 0)
-		(unit 1) (exclude_from_sim no) (in_bom yes) (on_board yes) (dnp no)
+		(unit 1) (exclude_from_sim no) (in_bom no) (on_board yes) (dnp no)
 		(property "Reference" "J5" (at 228.6 257.48 0)
 			(effects (font (size 1.27 1.27)) (justify left bottom)))
@@
 	(symbol (lib_id "gen:pads_3")
 		(at 741.68 210.82 0)
-		(unit 1) (exclude_from_sim no) (in_bom yes) (on_board yes) (dnp no)
+		(unit 1) (exclude_from_sim no) (in_bom no) (on_board yes) (dnp no)
 		(property "Reference" "J4" (at 731.52 199.06 0)
 			(effects (font (size 1.27 1.27)) (justify left bottom)))
