File: out/bluebuzz-rm2.kicad_sch (KiCad schematic)
At the start: 109 parts, among them J1 USB-C, J2 BAT, J3 SWD, J4 MOT, J5 TP, J6 PROBE, Q1 AO3400A, Q2 AO3400A, Q3 2N7002, SW1 PWR, U1 RP2350A, U10 USBLC6-2P6, U11 TPS22918DBVR, U2 BQ24074RGT, U20 DPS368, U21 DPS368, U22 DPS368, U23 DPS368, U24 DPS368, U3 TLV75533PDBV, U30 LSM6DS3TR-C, U5 TPS22918DBVR, U6 W25Q32JVUUIQ, U7 RM2, Y1 12MHz

Commit message: Configure GitHub Pages, add Pages link to README, export STEP without copper
Parts:
- removed C124: 100n, Capacitor_SMD:C_0402_1005Metric, symbol gen:C
- removed U24: DPS368, bluebuzz-rm2:DPS368_LGA-8, symbol gen:baro
- added C140: 100n, Capacitor_SMD:C_0402_1005Metric, symbol gen:C
- added U40: MP34DT05-A, bluebuzz-rm2:MP34DT05_HCLGA-4, symbol gen:pdm_mic
Connections:
- net 3V3_SYS: now also C140.1, U40.1 (VDD)
- net GND: now also C140.2, U40.2 (LR), U40.5 (GND)
- net PDM_DATA: now reaches U1.42 (GPIO28/PDM_DATA)
- net PDM_DATA: now also U40.4 (DOUT)
- net PDM_CLK: now reaches U1.43 (GPIO29/PDM_CLK)
- net PDM_CLK: now also U40.3 (CLK)
- net TAC_CS5: no longer names the net of U1.32 (GPIO20)
- no-connect marks 20 -> 19
Other:
- note added: "109 components / 72 nets / 6-layer. Bluetooth-audio vibrator controller: RP2350A + Raspberry Pi RM2 (CYW43439); USB-C, every other lead on back-side pads; BQ24074 charger with power path, a soft power latch (button, GPIO hold, USB), two low-side motor channels, 4 DPS368 barometers on the back (four corners and the centre, a tactile skin) on a switched 3.3 V rail, an IMU and a 1010 RGB status LED.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"
- note added: "14 — PDM MEMS microphone: MP34DT05-A (top-port)"
- note added: "Barometers): rubber poured over the array and pressure-cast (not vacuum: DPS368 p.43) so it fills"
- note added: "Four Infineon DPS368s on the BACK of the board in a diamond pattern (North U20, East U21, West"
- note added: "SNR, 122.5 dBSPL AOP) on the always-on 3.3 V rail. LR tied to GND selects the"
- note added: "SPI mode; SPI1 on GPIO10-12, one chip select each on GPIO0 and GPIO14-16. 100n at every sensor."
- note added: "ST MP34DT05TR-A top-port digital PDM MEMS microphone (3 x 4 x 1 mm HCLGA-4, 64 dB"
- note added: "U22, South U23), cast in soft elastomer after Tenzer, Jentoft & Howe 2014 (The Feel of MEMS"
- note added: "acoustic port needs no PCB hole."
- note added: "left-channel slot; CLK on GPIO29, DOUT on GPIO28 (PIO PDM state machine). Top"
- note added: "the ports; a load on the surface then reads as pressure. CSB low at power-up puts each sensor in"
- note removed: "109 components / 71 nets / 6-layer. Bluetooth-audio vibrator controller: RP2350A + Raspberry Pi RM2 (CYW43439); USB-C, every other lead on back-side pads; BQ24074 charger with power path, a soft power latch (button, GPIO hold, USB), two low-side motor channels, 5 DPS368 barometers on the back (four corners and the centre, a tactile skin) on a switched 3.3 V rail, an IMU and a 1010 RGB status LED.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"
- note removed: "Five Infineon DPS368s on the BACK of the board, one toward each corner and one in the centre,"
- note removed: "GPIO10-12, one chip select each on GPIO13-16 and 20. 100n at every sensor."
- note removed: "cast in soft elastomer after Tenzer, Jentoft & Howe 2014 (The Feel of MEMS Barometers): rubber"
- note removed: "on the surface then reads as pressure. CSB low at power-up puts each sensor in SPI mode; SPI1 on"
- note removed: "poured over the array and pressure-cast (not vacuum: DPS368 p.43) so it fills the ports; a load"
- moved on the sheet: C80, C81, C82, C83, C84, C85, C86, C87, C91, C92, C93, C94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
